File: Kicad/QsmeeScales.sch (KiCad schematic (older format))
At the start: 30 parts, among them J1 In-, J10 HX711 Load cell A/D, J11 7 Seg Display, J12 Load Cell, J2 In+, J3 Out+, J4 Out-, J5 P+, J6 P-, J7 B+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

Commit message: Tidy up schematic and add PDF
Parts:
- U1, U2: symbol Sensor:Load_cell -> QsmeeScales-rescue:Load_cell-Sensor
Other:
- note added: "LiPo 2S Ballance\nCharger"
- note removed: "LiPo Ballance\nCharger"
Changed lines of the file:
@@
 Title "Solar Powered Wheel Scales"
 Date "2019-09-27"
-Rev "1.0"
+Rev "1.01"
 Comp "QSMEE"
 Comment1 "QSMEE Solar Powered Wheel Loading Scales"
@@
 $EndComp
 $Comp
-L Sensor:Load_cell U1
+L QsmeeScales-rescue:Load_cell-Sensor U1
 U 1 1 5D955F8C
 P 10195 4255
@@
 $EndComp
 $Comp
-L Sensor:Load_cell U2
+L QsmeeScales-rescue:Load_cell-Sensor U2
 U 1 1 5D957F51
 P 10195 5685
@@
 	2510 2720 2510 2220
 Text Notes 2540 2485 0    25   ~ 0
-LiPo Ballance\nCharger
+LiPo 2S Ballance\nCharger
 Wire Notes Line
 	4450 6270 3750 6270
@@
 U 1 1 5DC7EDBC
 P 1435 2270
-F 0 "J2" H 1390 2285 50  0000 R CNN
+F 0 "J2" H 1420 2275 25  0000 R CNN
 F 1 "In+" H 1500 2355 50  0000 R CNN
 F 2 "" H 1435 2270 50  0001 C CNN
@@
 U 1 1 5DC800D8
 P 1430 2495
-F 0 "J1" H 1405 2495 50  0000 R CNN
+F 0 "J1" H 1415 2495 25  0000 R CNN
 F 1 "In-" H 1495 2450 50  0000 R CNN
 F 2 "" H 1430 2495 50  0001 C CNN
@@
 U 1 1 5DC816A3
 P 1765 2270
-F 0 "J3" H 1690 2275 50  0000 C CNN
+F 0 "J3" H 1725 2270 25  0000 C CNN
 F 1 "Out+" H 1725 2350 50  0000 C CNN
 F 2 "" H 1765 2270 50  0001 C CNN
@@
 U 1 1 5DC82563
 P 1765 2495
-F 0 "J4" H 1685 2530 50  0000 C CNN
+F 0 "J4" H 1725 2495 25  0000 C CNN
 F 1 "Out-" H 1720 2440 50  0000 C CNN
 F 2 "" H 1765 2495 50  0001 C CNN
@@
 U 1 1 5DC82F38
 P 2575 2330
-F 0 "J5" H 2500 2360 50  0000 R CNN
+F 0 "J5" H 2565 2335 25  0000 R CNN
 F 1 "P+" H 2630 2395 50  0000 R CNN
 F 2 "" H 2575 2330 50  0001 C CNN
@@
 U 1 1 5DC84027
 P 2585 2585
-F 0 "J6" H 2520 2620 50  0000 R CNN
+F 0 "J6" H 2570 2585 25  0000 R CNN
 F 1 "P-" H 2635 2530 50  0000 R CNN
 F 2 "" H 2585 2585 50  0001 C CNN
@@
 U 1 1 5DC84AD6
 P 2930 2325
-F 0 "J7" H 2850 2335 50  0000 C CNN
+F 0 "J7" H 2890 2325 25  0000 C CNN
 F 1 "B+" H 2940 2385 50  0000 C CNN
 F 2 "" H 2930 2325 50  0001 C CNN
@@
 U 1 1 5DC85523
 P 2945 2605
-F 0 "J9" H 2870 2620 50  0000 C CNN
+F 0 "J9" H 2910 2610 25  0000 C CNN
 F 1 "B-" H 2940 2555 50  0000 C CNN
 F 2 "" H 2945 2605 50  0001 C CNN
@@
 U 1 1 5DC86347
 P 2940 2480
-F 0 "J8" H 2860 2545 50  0000 C CNN
+F 0 "J8" H 2935 2510 25  0000 C CNN
 F 1 "BM" H 2865 2475 50  0000 C CNN
 F 2 "" H 2940 2480 50  0001 C CNN
